Commit message: Replace Encos placeholder motor specs with real Maxon HEJ values (URDF+MJCF)
Per electrical drawings-0623 + motor-ros FRAMEWORK_DESIGN.html (DS/AN sourced,
cross-validated <5%):
- armature (MJCF, HEJ50/70/90): 0.0056 / 0.0112 / 0.05 kg·m²
- peak torque (effort/ctrlrange): 30 / 62 / 140 N·m
- max speed @48V (URDF velocity): 21 / 17.8 / 10.4 rad/s
- MJCF actuators: <general>(placeholder kp=1) -> <motor ctrlrange=±peak> (match G1)
- EC_* (Encos) classes -> HEJ50/70/90; per-joint reassigned to correct model

kp/kd intentionally NOT in XML (computed in robot.py via omega_n=10Hz, zeta=2,
BeyondMimic arXiv 2508.08241). ROM/mass kept from CAD. Friction left at 0.
Verified: MuJoCo compiles (nu=31), all 31 joints match expected per-model values.

Co-Authored-By: Claude Opus 4.8 <noreply@anthropic.com>

File: src/holosoma/holosoma/data/robots/xhum_v2/xhum_v2_31dof.urdf (robot description, URDF)
Before this commit: robot xhum_v201, 34 links, 33 joints
Joints:
- joint head_pitch: limit lower=-0.785398 upper=0.785398 effort=12.0 velocity=100 -> lower=-0.785398 upper=0.785398 effort=30 velocity=21
- joint head_yaw: limit lower=-0.785398 upper=0.785398 effort=12.0 velocity=100 -> lower=-0.785398 upper=0.785398 effort=30 velocity=21
- joint left_ankle_pitch: limit lower=-0.872665 upper=0.872665 effort=36.0 velocity=100 -> lower=-0.872665 upper=0.872665 effort=62 velocity=17.8
- joint left_ankle_roll: limit lower=-0.261799 upper=0.261799 effort=36.0 velocity=100 -> lower=-0.261799 upper=0.261799 effort=30 velocity=21
- joint left_elbow: limit lower=-0.925025 upper=3.35103 effort=36.0 velocity=100 -> lower=-0.925025 upper=3.35103 effort=30 velocity=21
- joint left_hip_pitch: limit lower=-2.87979 upper=2.87979 effort=120.0 velocity=100 -> lower=-2.87979 upper=2.87979 effort=140 velocity=10.4
- joint left_hip_roll: limit lower=-1.0472 upper=1.29154 effort=120.0 velocity=100 -> lower=-1.0472 upper=1.29154 effort=62 velocity=17.8
- joint left_hip_yaw: limit lower=-2.53073 upper=2.53073 effort=60.0 velocity=100 -> lower=-2.53073 upper=2.53073 effort=140 velocity=10.4
- joint left_knee: limit lower=-0.0872665 upper=2.72271 effort=130.0 velocity=100 -> lower=-0.0872665 upper=2.72271 effort=140 velocity=10.4
- joint left_shoulder_pitch: limit lower=-4.01426 upper=1.5708 effort=36.0 velocity=100 -> lower=-4.01426 upper=1.5708 effort=62 velocity=17.8
- joint left_shoulder_roll: limit lower=-0.261799 upper=3.61283 effort=36.0 velocity=100 -> lower=-0.261799 upper=3.61283 effort=30 velocity=21
- joint left_shoulder_yaw: limit lower=-2.53073 upper=2.53073 effort=36.0 velocity=100 -> lower=-2.53073 upper=2.53073 effort=30 velocity=21
- joint left_wrist_pitch: limit lower=-1.0472 upper=1.0472 effort=12.0 velocity=100 -> lower=-1.0472 upper=1.0472 effort=30 velocity=21
- joint left_wrist_roll: limit lower=-2.53073 upper=2.53073 effort=36.0 velocity=100 -> lower=-2.53073 upper=2.53073 effort=30 velocity=21
- joint left_wrist_yaw: limit lower=-1.39626 upper=1.39626 effort=12.0 velocity=100 -> lower=-1.39626 upper=1.39626 effort=30 velocity=21
- joint right_ankle_pitch: limit lower=-0.872665 upper=0.872665 effort=36.0 velocity=100 -> lower=-0.872665 upper=0.872665 effort=62 velocity=17.8
- joint right_ankle_roll: limit lower=-0.261799 upper=0.261799 effort=36.0 velocity=100 -> lower=-0.261799 upper=0.261799 effort=30 velocity=21
- joint right_elbow: limit lower=-0.925025 upper=3.35103 effort=36.0 velocity=100 -> lower=-0.925025 upper=3.35103 effort=30 velocity=21
- joint right_hip_pitch: limit lower=-2.87979 upper=2.87979 effort=120.0 velocity=100 -> lower=-2.87979 upper=2.87979 effort=140 velocity=10.4
- joint right_hip_roll: limit lower=-1.29154 upper=1.0472 effort=120.0 velocity=100 -> lower=-1.29154 upper=1.0472 effort=62 velocity=17.8
- joint right_hip_yaw: limit lower=-2.53073 upper=2.53073 effort=60.0 velocity=100 -> lower=-2.53073 upper=2.53073 effort=140 velocity=10.4
- joint right_knee: limit lower=-0.0872665 upper=2.72271 effort=130.0 velocity=100 -> lower=-0.0872665 upper=2.72271 effort=140 velocity=10.4
- joint right_shoulder_pitch: limit lower=-4.01426 upper=1.5708 effort=36.0 velocity=100 -> lower=-4.01426 upper=1.5708 effort=62 velocity=17.8
- joint right_shoulder_roll: limit lower=-3.61283 upper=0.261799 effort=36.0 velocity=100 -> lower=-3.61283 upper=0.261799 effort=30 velocity=21
- joint right_shoulder_yaw: limit lower=-2.53073 upper=2.53073 effort=36.0 velocity=100 -> lower=-2.53073 upper=2.53073 effort=30 velocity=21
- joint right_wrist_pitch: limit lower=-1.0472 upper=1.0472 effort=12.0 velocity=100 -> lower=-1.0472 upper=1.0472 effort=30 velocity=21
- joint right_wrist_roll: limit lower=-2.53073 upper=2.53073 effort=36.0 velocity=100 -> lower=-2.53073 upper=2.53073 effort=30 velocity=21
- joint right_wrist_yaw: limit lower=-1.39626 upper=1.39626 effort=12.0 velocity=100 -> lower=-1.39626 upper=1.39626 effort=30 velocity=21
- joint waist_pitch: limit lower=-0.436332 upper=0.610865 effort=75.0 velocity=100 -> lower=-0.436332 upper=0.610865 effort=62 velocity=17.8
- joint waist_roll: limit lower=-0.698132 upper=0.698132 effort=60.0 velocity=100 -> lower=-0.698132 upper=0.698132 effort=62 velocity=17.8
- joint waist_yaw: limit lower=-1.5708 upper=1.5708 effort=75.0 velocity=100 -> lower=-1.5708 upper=1.5708 effort=62 velocity=17.8

Commit message: Fix xhum_v2 IsaacSim load: URDF root link + disabled-gantry crash
Two fixes found via smoke test (exp:xhum_v2-31dof-fast-sac on IsaacSim):
1. URDF: removed 'world' link + 'floating_humanoid' floating joint so 'humanoid'
   is the root link. The world+floating-joint structure made IsaacLab fail to
   enumerate the articulation joints (resolve_matching_names: Available strings []).
   Now matches G1 convention (root = base link, sim adds the floating base).
2. virtual_gantry.create_virtual_gantry: when gantry is DISABLED, no longer raises
   if no attachment body matches the hardcoded name list — returns a no-op gantry
   (body_link_id unused when disabled). Lets robots with non-standard body names
   (xhum_v2: humanoid/waist_bridge_2_01/chest_2_01) train.

Smoke test: 64 envs, reached iter 294/50000 @ ~14 it/s, rewards updating, clean stop.

Co-Authored-By: Claude Opus 4.8 <noreply@anthropic.com>

File: src/holosoma/holosoma/data/robots/xhum_v2/xhum_v2_31dof.urdf (robot description, URDF)
Before this commit: robot xhum_v201, 34 links, 33 joints
Links:
- removed link world
Joints:
- removed joint floating_humanoid

Commit message: Fix xhum_v2 kneel collapse: add foot contact points for feet_phase/feet_ori
xhum_v2 的 fast-sac 策略训练到 ~21k 步坍缩成稳定深跪(根高~0.5m,膝~2.4rad),
始终学不会走。根因:foot_height_name/foot_body_name 指向 onshape 导出的原始
`foot` body——其原点离鞋底 ~8cm、坐标系非语义(z 轴偏竖直 ~87°)。导致:
- feet_phase(迈步奖励)因脚高恒有 ~8cm 偏置而拿不到分(raw ~10x 低于 G1);
- feet_ori(脚朝向惩罚)因非语义帧把平脚算成大幅倾斜而恒重罚(~6x G1)。
于是"站立行走"净回报低于"稳定跪",策略坍缩进跪姿(已交叉验证排除腿软/增益问题:
前 20k 稳站 0.83m、稳定跪 862 步说明执行器有力支撑、G1 零动作可站满)。

修复(照 G1 做法):在 foot_2/foot(双踝之下末端脚连杆)各加贴鞋底、默认平脚时
朝向对齐世界竖直的 left/right_foot_contact_point(FK 算偏移/rpy,落点距鞋底
<1mm、z 轴竖直);foot_height_name/foot_body_name/key_bodies 指向接触点;
body_names +2、num_bodies 34。

冒烟验证(默认姿态):feet_phase 0.914(原 ~0.1-0.45)、penalty_feet_ori 0.092
(原 ~1.0+)。需重训验证是否能学会行走。

Co-Authored-By: Claude Opus 4.8 <noreply@anthropic.com>

File: src/holosoma/holosoma/data/robots/xhum_v2/xhum_v2_31dof.urdf (robot description, URDF)
Before this commit: robot xhum_v201, 33 links, 32 joints
Links:
- added link left_foot_contact_point, mass 0.001; visual sphere radius=0.005
- added link right_foot_contact_point, mass 0.001; visual sphere radius=0.005
Joints:
- added joint left_foot_contact_point: type fixed, parent foot_2, child left_foot_contact_point, origin xyz=-0.0644 0.0 0.0054 rpy=1.5292 0.1474 1.5453
- added joint right_foot_contact_point: type fixed, parent foot, child right_foot_contact_point, origin xyz=-0.0643 0.0 0.0054 rpy=1.5292 -0.1474 1.5963

Commit message: Fix xhum_v2 leg/arm motor spec per electrical drawing
By aligning the electrical-drawing 4-bus daisy-chain order to URDF joint
order, found hip_roll/hip_yaw motor types swapped and shoulder_roll under-spec'd:
- hip_roll:      HEJ70 -> HEJ90 (effort 62->140, vel 17.8->10.4, armature 0.0112->0.05, kp 44.2->197.4, kd 2.81->12.57)
- hip_yaw:       HEJ90 -> HEJ70 (reverse of above)
- shoulder_roll: HEJ50 -> HEJ70 (effort 30->62, vel 21->17.8, armature 0.0056->0.0112, kp 22.1->44.2, kd 1.41->2.81)

Synced across robot.py (dof_effort/vel/armature lists + stiffness/damping),
URDF <limit effort/velocity>, and MJCF (joint class + motor ctrlrange).
Counts verified HEJ90x6 / HEJ70x11 / HEJ50x14; MuJoCo compiles clean.

Co-Authored-By: Claude Opus 4.8 (1M context) <noreply@anthropic.com>

File: src/holosoma/holosoma/data/robots/xhum_v2/xhum_v2_31dof.urdf (robot description, URDF)
Before this commit: robot xhum_v201, 35 links, 34 joints
Joints:
- joint left_hip_roll: limit lower=-1.0472 upper=1.29154 effort=62 velocity=17.8 -> lower=-1.0472 upper=1.29154 effort=140 velocity=10.4
- joint left_hip_yaw: limit lower=-2.53073 upper=2.53073 effort=140 velocity=10.4 -> lower=-2.53073 upper=2.53073 effort=62 velocity=17.8
- joint left_shoulder_roll: limit lower=-0.261799 upper=3.61283 effort=30 velocity=21 -> lower=-0.261799 upper=3.61283 effort=62 velocity=17.8
- joint right_hip_roll: limit lower=-1.29154 upper=1.0472 effort=62 velocity=17.8 -> lower=-1.29154 upper=1.0472 effort=140 velocity=10.4
- joint right_hip_yaw: limit lower=-2.53073 upper=2.53073 effort=140 velocity=10.4 -> lower=-2.53073 upper=2.53073 effort=62 velocity=17.8
- joint right_shoulder_roll: limit lower=-3.61283 upper=0.261799 effort=30 velocity=21 -> lower=-3.61283 upper=0.261799 effort=62 velocity=17.8
