Commit message: Replace xhum_v2 assets with v2.01 canonical baseline (path-only adaptation)
Swap the old (frame-unaligned, hand-patched) xhum_v2 URDF/MJCF/meshes for the
v2.01 canonical baseline (commit 0a6343d). New files are byte-identical to the
v2.01 baseline except holosoma mesh-path conventions:
- URDF: package://xhum/meshes/xhum2/ -> meshes/
- MJCF: meshdir="assets/" -> "./meshes/" ; file="merged/X" -> file="X"
No geometry/motor/frame edits here (those are upstream in v2.01).

Also drops the transitional hum2.0_dev_v2.01_20260622/ working-tree copy
(33MB; preserved in history 0a6343d, recover via git checkout 0a6343d -- <path>).

Step 2 of 4 (verified: xhum_v2 differs from v2.01 baseline only in mesh paths).

Co-Authored-By: Claude Opus 4.8 (1M context) <noreply@anthropic.com>

File: src/holosoma/holosoma/data/robots/xhum_v2/xhum_v2_31dof.urdf (robot description, URDF)
Before this commit: robot xhum_v201, 35 links, 34 joints
Links:
- removed link ankle
- removed link arm_j2_left
- removed link arm_j2_right
- removed link arm_j3
- removed link arm_j3_2
- removed link arm_j4
- removed link arm_j4_l
- removed link arm_j5
- removed link arm_j5_2
- removed link arm_j5_output
- removed link arm_j5_output_2
- removed link arm_j7_l
- removed link arm_j7_r
- removed link calf
- removed link chest_2_01
- removed link foot
- removed link foot_2
- removed link hand_output
- removed link hand_output_2
- removed link hip_yaw_left
- removed link hip_yaw_left_2
- removed link hiproll_motor_l
- removed link hiproll_motor_r
- removed link left_foot_contact_point
- removed link left_knee
- removed link neck_j1_motor
- removed link right_ankle
- removed link right_calf
- removed link right_foot_contact_point
- removed link right_knee
- removed link waist_bridge_2_01
- removed link waist_pitch_motor
- removed link waist_roll_motor
- added link head_yaw_link, mass 0.697313; collision capsule length=0.0388498 radius=0.0285228; visual mesh filename=meshes/converted_neck_j1_motor_visual.stl
- added link left_ankle_pitch_link, mass 1.45033; collision capsule length=0.0886334 radius=0.0400865; visual mesh filename=meshes/converted_ankle_roll_motor_l_visual.stl
- added link left_ankle_roll_link, mass 0.778414; visual mesh filename=meshes/converted_foot_visual.stl
- added link left_elbow_link, mass 0.809734; collision capsule length=0.0917666 radius=0.0322981; visual mesh filename=meshes/converted_arm_j5_r_2_visual.stl
- added link left_foot, mass 1e-06; collision capsule length=0.214 radius=0.01; collision capsule length=0.214 radius=0.01
- added link left_hip_pitch_link, mass 2.87104; collision capsule length=0.06 radius=0.04; visual mesh filename=meshes/converted_hiproll_motor_l_visual.stl
- added link left_hip_roll_link, mass 0.633113; collision capsule length=0.095854 radius=0.0386053; visual mesh filename=meshes/converted_hip_yaw_left_visual.stl
- added link left_hip_yaw_link, mass 4.55978; collision capsule length=0.217152 radius=0.0443949; visual mesh filename=meshes/converted_left_knee_visual.stl
- added link left_knee_link, mass 2.43041; collision capsule length=0.205942 radius=0.0439052; visual mesh filename=meshes/converted_calf_l_visual.stl
- added link left_shoulder_pitch_link, mass 1.52519; collision capsule length=0.0594946 radius=0.0409161; visual mesh filename=meshes/converted_arm_j2_l_visual.stl
- added link left_shoulder_roll_link, mass 0.933252; collision capsule length=0.130169 radius=0.0354106; visual mesh filename=meshes/converted_arm_j3_r_2_visual.stl
- added link left_shoulder_yaw_link, mass 0.900942; collision capsule length=0.0776256 radius=0.0293826; visual mesh filename=meshes/converted_arm_j4_l_visual.stl
- added link left_wrist_pitch_link, mass 0.665084; collision capsule length=0.0366386 radius=0.0274352; visual mesh filename=meshes/converted_arm_j7_visual.stl
- added link left_wrist_roll_link, mass 1.34224; collision capsule length=0.0915576 radius=0.038822; visual mesh filename=meshes/converted_arm_j6_r_2_visual.stl
- added link left_wrist_yaw_link, mass 0.233204; collision capsule length=0.1009476 radius=0.0262118; visual mesh filename=meshes/converted_hand_output_2_visual.stl
- added link pelvis, mass 7.13645; collision capsule length=0.203226 radius=0.0568495; visual mesh filename=meshes/converted_waist_bridge_2_visual.stl
- added link right_ankle_pitch_link, mass 1.46466; collision capsule length=0.088689 radius=0.0400441; visual mesh filename=meshes/converted_ankle_roll_motor_r_visual.stl
- added link right_ankle_roll_link, mass 0.778414; visual mesh filename=meshes/converted_foot_2_visual.stl
- added link right_elbow_link, mass 0.809734; collision capsule length=0.0917884 radius=0.0322991; visual mesh filename=meshes/converted_arm_j5_r_visual.stl
- added link right_foot, mass 1e-06; collision capsule length=0.214 radius=0.01; collision capsule length=0.214 radius=0.01
- added link right_hip_pitch_link, mass 2.87137; collision capsule length=0.06 radius=0.04; visual mesh filename=meshes/converted_hiproll_motor_r_visual.stl
- added link right_hip_roll_link, mass 0.633113; collision capsule length=0.095854 radius=0.0386053; visual mesh filename=meshes/converted_hip_yaw_left_2_visual.stl
- added link right_hip_yaw_link, mass 4.55417; collision capsule length=0.216686 radius=0.0443938; visual mesh filename=meshes/converted_right_knee_visual.stl
- added link right_knee_link, mass 2.43041; collision capsule length=0.206594 radius=0.0439104; visual mesh filename=meshes/converted_calf_r_visual.stl
- added link right_shoulder_pitch_link, mass 1.53789; collision capsule length=0.0594816 radius=0.0408814; visual mesh filename=meshes/converted_arm_j2_r_visual.stl
- added link right_shoulder_roll_link, mass 0.933252; collision capsule length=0.1301812 radius=0.0354082; visual mesh filename=meshes/converted_arm_j3_r_visual.stl
- added link right_shoulder_yaw_link, mass 0.903604; collision capsule length=0.0777274 radius=0.0293217; visual mesh filename=meshes/converted_arm_j4_r_visual.stl
- added link right_wrist_pitch_link, mass 0.665084; collision capsule length=0.0366638 radius=0.0274302; visual mesh filename=meshes/converted_arm_j7_r_visual.stl
- added link right_wrist_roll_link, mass 1.34224; collision capsule length=0.0916406 radius=0.0387983; visual mesh filename=meshes/converted_arm_j6_r_visual.stl
- added link right_wrist_yaw_link, mass 0.233204; collision capsule length=0.1009476 radius=0.0262118; visual mesh filename=meshes/converted_hand_output_visual.stl
- added link torso_link, mass 14.5548; collision capsule length=0.1820688 radius=0.110801; visual mesh filename=meshes/converted_chest_2_01_visual.stl
- added link waist_pitch_link, mass 0.282742; collision capsule length=0.0855778 radius=0.0284277; visual mesh filename=meshes/converted_waist_yaw_visual.stl
- added link waist_roll_link, mass 1.75074; visual mesh filename=meshes/converted_waist_pitch_visual.stl
Joints:
- removed joint humanoid2waist_bridge_2_01_fixed
- removed joint left_foot_contact_point
- removed joint right_foot_contact_point
- added joint humanoid2pelvis_fixed: type fixed, parent humanoid, child pelvis, origin xyz=0.0 0.0 0.0 rpy=0.0 0.0 0.0
- added joint left_ankle_roll_link2left_foot_fixed: type fixed, parent left_ankle_roll_link, child left_foot, origin xyz=-0.058 0.0 0.0 rpy=-0.0 1.5707963267948966 0.0
- added joint right_ankle_roll_link2right_foot_fixed: type fixed, parent right_ankle_roll_link, child right_foot, origin xyz=-0.058 0.0 0.0 rpy=-0.0 1.5707963267948966 0.0
- joint head_pitch: limit lower=-0.785398 upper=0.785398 effort=30 velocity=21 -> lower=-0.785398 upper=0.785398 effort=30.0 velocity=100; parent neck_j1_motor -> head_yaw_link
- joint head_yaw: axis 0.0 0.0 1.0 -> 0.0 0.0 -1.0; child neck_j1_motor -> head_yaw_link; limit lower=-0.785398 upper=0.785398 effort=30 velocity=21 -> lower=-0.785398 upper=0.785398 effort=30.0 velocity=100; parent chest_2_01 -> torso_link
- joint left_ankle_pitch: child ankle -> left_ankle_pitch_link; limit lower=-0.872665 upper=0.872665 effort=62 velocity=17.8 -> lower=-0.872665 upper=0.872665 effort=62.0 velocity=100; parent calf -> left_knee_link
- joint left_ankle_roll: child foot_2 -> left_ankle_roll_link; limit lower=-0.261799 upper=0.261799 effort=30 velocity=21 -> lower=-0.261799 upper=0.261799 effort=30.0 velocity=100; parent ankle -> left_ankle_pitch_link
- joint left_elbow: child arm_j5_2 -> left_elbow_link; limit lower=-0.925025 upper=3.35103 effort=30 velocity=21 -> lower=-0.925025 upper=3.35103 effort=30.0 velocity=100; parent arm_j4_l -> left_shoulder_yaw_link
- joint left_hip_pitch: child hiproll_motor_l -> left_hip_pitch_link; limit lower=-2.87979 upper=2.87979 effort=140 velocity=10.4 -> lower=-2.87979 upper=2.87979 effort=140.0 velocity=100; parent waist_bridge_2_01 -> pelvis
- joint left_hip_roll: child hip_yaw_left -> left_hip_roll_link; limit lower=-1.0472 upper=1.29154 effort=140 velocity=10.4 -> lower=-1.0472 upper=1.29154 effort=140.0 velocity=100; parent hiproll_motor_l -> left_hip_pitch_link
- joint left_hip_yaw: child left_knee -> left_hip_yaw_link; limit lower=-2.53073 upper=2.53073 effort=62 velocity=17.8 -> lower=-2.53073 upper=2.53073 effort=62.0 velocity=100; parent hip_yaw_left -> left_hip_roll_link
- joint left_knee: child calf -> left_knee_link; limit lower=-0.0872665 upper=2.72271 effort=140 velocity=10.4 -> lower=-0.0872665 upper=2.72271 effort=140.0 velocity=100; parent left_knee -> left_hip_yaw_link
- joint left_shoulder_pitch: child arm_j2_left -> left_shoulder_pitch_link; limit lower=-4.01426 upper=1.5708 effort=62 velocity=17.8 -> lower=-4.01426 upper=1.5708 effort=62.0 velocity=100; parent chest_2_01 -> torso_link
- joint left_shoulder_roll: child arm_j3_2 -> left_shoulder_roll_link; limit lower=-0.261799 upper=3.61283 effort=62 velocity=17.8 -> lower=-0.261799 upper=3.61283 effort=62.0 velocity=100; parent arm_j2_left -> left_shoulder_pitch_link
- joint left_shoulder_yaw: child arm_j4_l -> left_shoulder_yaw_link; limit lower=-2.53073 upper=2.53073 effort=30 velocity=21 -> lower=-2.53073 upper=2.53073 effort=30.0 velocity=100; parent arm_j3_2 -> left_shoulder_roll_link
- joint left_wrist_pitch: child arm_j7_l -> left_wrist_pitch_link; limit lower=-1.0472 upper=1.0472 effort=30 velocity=21 -> lower=-1.0472 upper=1.0472 effort=30.0 velocity=100; parent arm_j5_output_2 -> left_wrist_roll_link
- joint left_wrist_roll: child arm_j5_output_2 -> left_wrist_roll_link; limit lower=-2.53073 upper=2.53073 effort=30 velocity=21 -> lower=-2.53073 upper=2.53073 effort=30.0 velocity=100; parent arm_j5_2 -> left_elbow_link
- joint left_wrist_yaw: child hand_output_2 -> left_wrist_yaw_link; limit lower=-1.39626 upper=1.39626 effort=30 velocity=21 -> lower=-1.39626 upper=1.39626 effort=30.0 velocity=100; parent arm_j7_l -> left_wrist_pitch_link
- joint right_ankle_pitch: child right_ankle -> right_ankle_pitch_link; limit lower=-0.872665 upper=0.872665 effort=62 velocity=17.8 -> lower=-0.872665 upper=0.872665 effort=62.0 velocity=100; parent right_calf -> right_knee_link
- joint right_ankle_roll: child foot -> right_ankle_roll_link; limit lower=-0.261799 upper=0.261799 effort=30 velocity=21 -> lower=-0.261799 upper=0.261799 effort=30.0 velocity=100; parent right_ankle -> right_ankle_pitch_link
- joint right_elbow: child arm_j5 -> right_elbow_link; limit lower=-0.925025 upper=3.35103 effort=30 velocity=21 -> lower=-0.925025 upper=3.35103 effort=30.0 velocity=100; parent arm_j4 -> right_shoulder_yaw_link
- joint right_hip_pitch: child hiproll_motor_r -> right_hip_pitch_link; limit lower=-2.87979 upper=2.87979 effort=140 velocity=10.4 -> lower=-2.87979 upper=2.87979 effort=140.0 velocity=100; parent waist_bridge_2_01 -> pelvis
- joint right_hip_roll: child hip_yaw_left_2 -> right_hip_roll_link; limit lower=-1.29154 upper=1.0472 effort=140 velocity=10.4 -> lower=-1.29154 upper=1.0472 effort=140.0 velocity=100; parent hiproll_motor_r -> right_hip_pitch_link
- joint right_hip_yaw: child right_knee -> right_hip_yaw_link; limit lower=-2.53073 upper=2.53073 effort=62 velocity=17.8 -> lower=-2.53073 upper=2.53073 effort=62.0 velocity=100; parent hip_yaw_left_2 -> right_hip_roll_link
- joint right_knee: child right_calf -> right_knee_link; limit lower=-0.0872665 upper=2.72271 effort=140 velocity=10.4 -> lower=-0.0872665 upper=2.72271 effort=140.0 velocity=100; parent right_knee -> right_hip_yaw_link
- joint right_shoulder_pitch: child arm_j2_right -> right_shoulder_pitch_link; limit lower=-4.01426 upper=1.5708 effort=62 velocity=17.8 -> lower=-4.01426 upper=1.5708 effort=62.0 velocity=100; parent chest_2_01 -> torso_link
- joint right_shoulder_roll: child arm_j3 -> right_shoulder_roll_link; limit lower=-3.61283 upper=0.261799 effort=62 velocity=17.8 -> lower=-3.61283 upper=0.261799 effort=62.0 velocity=100; parent arm_j2_right -> right_shoulder_pitch_link
- joint right_shoulder_yaw: child arm_j4 -> right_shoulder_yaw_link; limit lower=-2.53073 upper=2.53073 effort=30 velocity=21 -> lower=-2.53073 upper=2.53073 effort=30.0 velocity=100; parent arm_j3 -> right_shoulder_roll_link
- joint right_wrist_pitch: child arm_j7_r -> right_wrist_pitch_link; limit lower=-1.0472 upper=1.0472 effort=30 velocity=21 -> lower=-1.0472 upper=1.0472 effort=30.0 velocity=100; parent arm_j5_output -> right_wrist_roll_link
- joint right_wrist_roll: child arm_j5_output -> right_wrist_roll_link; limit lower=-2.53073 upper=2.53073 effort=30 velocity=21 -> lower=-2.53073 upper=2.53073 effort=30.0 velocity=100; parent arm_j5 -> right_elbow_link
- joint right_wrist_yaw: child hand_output -> right_wrist_yaw_link; limit lower=-1.39626 upper=1.39626 effort=30 velocity=21 -> lower=-1.39626 upper=1.39626 effort=30.0 velocity=100; parent arm_j7_r -> right_wrist_pitch_link
- joint waist_pitch: child waist_roll_motor -> waist_pitch_link; limit lower=-0.436332 upper=0.610865 effort=62 velocity=17.8 -> lower=-0.436332 upper=0.610865 effort=62.0 velocity=100; parent waist_pitch_motor -> waist_roll_link
- joint waist_roll: child waist_pitch_motor -> waist_roll_link; limit lower=-0.698132 upper=0.698132 effort=62 velocity=17.8 -> lower=-0.698132 upper=0.698132 effort=62.0 velocity=100; parent waist_bridge_2_01 -> pelvis
- joint waist_yaw: child chest_2_01 -> torso_link; limit lower=-1.5708 upper=1.5708 effort=62 velocity=17.8 -> lower=-1.5708 upper=1.5708 effort=62.0 velocity=100; parent waist_roll_motor -> waist_pitch_link

Commit message: Sync frame-aligned xhum_v2 URDF + visual meshes from v2.01 regen
Pull the colleague's regenerated v2.01 (humanoid_internal) into holosoma:
- URDF: replace xhum_v2_31dof.urdf with the convert_urdf-fixed version.
  base-x is now forward (hips at Y=±0.117, was X), matching the already-
  aligned MJCF. Mesh paths adapted package://xhum/meshes/xhum2/ -> meshes/.
- Meshes: update the 32 converted_*_visual.stl (visual only) to match.

Verified before sync (no other change needed):
- MJCF(.xml) physics already identical to new output.xml (body pose, joint
  axis/range, inertia, collision geoms, self-collision excludes: 0 diff);
  left as-is to keep the motor/HEJ actuator adaptation (general->motor).
- masses 63.683kg total, 0 per-link diff across old/new URDF + MJCF.
- joint axes vs symmetry flip-sign table: 31/31 consistent.

Co-Authored-By: Claude Opus 4.8 (1M context) <noreply@anthropic.com>

File: src/holosoma/holosoma/data/robots/xhum_v2/xhum_v2_31dof.urdf (robot description, URDF)
Before this commit: robot converted_robot, 35 links, 34 joints
Joints:
- joint head_pitch: axis 0.0 0.0 1.0 -> 0.0 1.0 0.0; origin xyz=-0.03815 0.0 -0.046 rpy=-3.141592653589793 -1.5707963267948966 0.0 -> xyz=-1.2803381e-10 -0.03815 0.046 rpy=0.0 0.0 0.0
- joint head_yaw: axis 0.0 0.0 -1.0 -> -8.952402789524028e-34 -4.0178667401786675e-17 1.0; origin xyz=0.0 0.0 -0.307 rpy=0.0 0.0 1.5707963267948966 -> xyz=0.0 -1.233485e-17 0.307 rpy=0.0 0.0 0.0
- joint left_ankle_pitch: axis 0.0 0.0 -1.0 -> 9.000588599993941e-07 0.9999999999993268 7.326174399995069e-07; origin xyz=0.0845237 -0.181262 0.00495 rpy=0.0 0.0 -2.879793683130459 -> xyz=-2.7372142e-07 -0.0049498541 -0.20000043 rpy=0.0 0.0 0.0
- joint left_ankle_roll: axis 0.0 0.0 -1.0 -> 0.9999999999995153 -9.000585599995637e-07 -3.993358099998065e-07; origin xyz=-0.0440453 0.0876837 0.0336 rpy=-1.5707963267948968 0.0 -1.3962627673627896 -> xyz=0.02814991 -0.033599957 -0.094000028 rpy=0.0 0.0 0.0
- joint left_ankle_roll_link2left_foot_fixed: origin xyz=-0.058 0.0 0.0 rpy=-0.0 1.5707963267948966 0.0 -> xyz=-2.3161439e-08 4.2365282e-08 -0.058000001 rpy=0.0 0.0 0.0
- joint left_elbow: axis 0.0 0.0 1.0 -> 0.0 1.0 0.0; origin xyz=-0.0494702 -0.0135849 -0.078 rpy=2.617993281776241 -1.5707963267948966 0.0 -> xyz=0.036499989 -0.036049978 -0.078 rpy=0.0 0.0 0.0
- joint left_hip_pitch: axis 0.0 0.0 -1.0 -> 8.437658953288307e-07 0.8660254654694117 -0.49999989315776544; origin xyz=0.116524 0.05 -0.087275 rpy=-1.040543549740843 -0.15095625512435595 1.4828593469166491 -> xyz=-0.049999999 0.116524 -0.087275 rpy=0.0 0.0 0.0
- joint left_hip_roll: axis 0.0 0.0 -1.0 -> 0.999999999999591 -8.952151589517855e-07 1.291326512912737e-07; origin xyz=-0.0547845 0.0512656 -0.078 rpy=-2.9670597689824123 -1.5707963267948966 0.0 -> xyz=0.04505007 0.03754996 -0.090961502 rpy=0.0 0.0 0.0
- joint left_hip_yaw: axis 0.0 0.0 1.0 -> -1.363451499999625e-07 -7.290808999997995e-07 0.9999999999997249; origin xyz=-0.0455 -0.0788083 0.04505 rpy=-1.5707963267948966 0.0 -0.5235993718135523 -> xyz=-0.045049988 5.7724054e-08 -0.090999995 rpy=0.0 0.0 0.0
- joint left_knee: axis 0.0 0.0 -1.0 -> 9.000514399993959e-07 0.9999999999993288 7.2992522999951e-07; origin xyz=-0.03855 -0.03 -0.19555 rpy=1.5707963267948966 0.43633306990197296 1.5707963267948966 -> xyz=-0.029999938 0.038550169 -0.19554998 rpy=0.0 0.0 0.0
- joint left_shoulder_pitch: axis 0.0 0.0 -1.0 -> -2.119336687940619e-17 0.9396927646529906 0.3420197480538503; origin xyz=0.0 0.152633 -0.258339 rpy=0.0 -1.2217309121094393 1.5707963267948966 -> xyz=0.0 0.152633 0.258339 rpy=0.0 0.0 0.0
- joint left_shoulder_roll: axis 0.0 0.0 -1.0 -> 1.0 0.0 0.0; origin xyz=0.0165606 0.03995 -0.076 rpy=-1.5707963267948966 -1.2217309121094393 3.141592653589793 -> xyz=0.03995 0.077080702 0.010431625 rpy=0.0 0.0 0.0
- joint left_shoulder_yaw: origin xyz=0.0 -0.15135 0.038 rpy=1.5707963267948966 -0.5235993718135523 -3.141592653589793 -> xyz=-0.038 0.0 -0.15135 rpy=0.0 0.0 0.0
- joint left_wrist_pitch: axis 0.0 0.0 1.0 -> -3.484140899999884e-17 0.9999999999999667 2.579144899999914e-07; origin xyz=0.0372391 -0.0215 -0.1665 rpy=0.5235993718135523 1.5707963267948966 0.0 -> xyz=0.1665 0.043000008 -1.5784863e-08 rpy=0.0 0.0 0.0
- joint left_wrist_roll: axis 0.0 0.0 -1.0 -> 1.0 -4.4377618e-18 1.5252148e-08; origin xyz=0.0 0.12035 0.036 rpy=-1.5707963267948966 -1.047197210609006 3.141592653589793 -> xyz=0.12035 0.036 6.9388939e-18 rpy=0.0 0.0 0.0
- joint left_wrist_yaw: axis 0.0 0.0 -1.0 -> 2.199174199999929e-17 -2.545584399999917e-07 0.9999999999999676; origin xyz=0.0 -0.03315 -0.043 rpy=1.5707963267948966 0.0 -3.141592653589793 -> xyz=2.2272069e-18 -0.043000008 0.033149989 rpy=0.0 0.0 0.0
- joint right_ankle_pitch: axis 0.0 0.0 1.0 -> 9.109927399993883e-07 0.9999999999993285 -7.16323209999519e-07; origin xyz=0.0845237 0.181262 0.00495 rpy=0.0 0.0 2.879793683130459 -> xyz=-3.1991704e-07 0.0049498544 -0.20000043 rpy=0.0 0.0 0.0
- joint right_ankle_roll: axis 0.0 0.0 -1.0 -> 0.9999999999993523 -9.1099322999941e-07 -6.821777899995582e-07; origin xyz=-0.0440453 -0.0876837 0.0336 rpy=1.5707963267948968 0.0 1.3962627673627896 -> xyz=0.028149945 0.033599907 -0.094000035 rpy=0.0 0.0 0.0
- joint right_ankle_roll_link2right_foot_fixed: origin xyz=-0.058 0.0 0.0 rpy=-0.0 1.5707963267948966 0.0 -> xyz=-3.956635e-08 -4.1674658e-08 -0.058 rpy=0.0 0.0 0.0
- joint right_elbow: axis 0.0 0.0 -1.0 -> 0.0 1.0 0.0; origin xyz=0.0129702 -0.0496349 -0.078 rpy=-0.5235993718135523 -1.5707963267948966 0.0 -> xyz=0.036499963 0.036049994 -0.078 rpy=0.0 0.0 0.0
- joint right_hip_pitch: axis 0.0 0.0 1.0 -> 8.437658953288307e-07 0.8660254654694117 0.49999989315776544; origin xyz=-0.116524 0.05 -0.087275 rpy=1.040543549740843 0.15095625512435618 1.4828593469166491 -> xyz=-0.05 -0.116524 -0.087275 rpy=0.0 0.0 0.0
- joint right_hip_roll: axis 0.0 0.0 -1.0 -> 0.999999999999589 -8.952151589517838e-07 -1.435563514355045e-07; origin xyz=-0.0339467 -0.0669113 -0.078 rpy=-0.17453288460738095 1.5707963267948966 0.0 -> xyz=0.04504995 -0.037550041 -0.090961513 rpy=0.0 0.0 0.0
- joint right_hip_yaw: axis 0.0 0.0 1.0 -> 1.363451499999625e-07 7.290808999997995e-07 0.9999999999997249; origin xyz=0.0455 -0.0788083 0.04505 rpy=1.5707963267948966 0.0 -2.617993281776241 -> xyz=-0.045050012 2.1798124e-08 -0.090999983 rpy=0.0 0.0 0.0
- joint right_knee: axis 0.0 0.0 1.0 -> 9.115179999993793e-07 0.999999999999319 -7.288771399995036e-07; origin xyz=-0.03855 0.03 -0.19555 rpy=-1.5707963267948966 0.43633306990197296 -1.5707963267948966 -> xyz=-0.030000062 -0.038550115 -0.19554997 rpy=0.0 0.0 0.0
- joint right_shoulder_pitch: axis 0.0 0.0 1.0 -> 0.0 0.9396923976377319 -0.3420207564196225; origin xyz=0.0 -0.152633 -0.258339 rpy=1.2217298123263818 0.0 3.141592653589793 -> xyz=0.0 -0.152633 0.258339 rpy=0.0 0.0 0.0
- joint right_shoulder_roll: axis 0.0 0.0 -1.0 -> 1.0 0.0 0.0; origin xyz=0.03995 0.0165606 -0.076 rpy=-1.5707963267948966 1.2217298123263816 1.5707963267948966 -> xyz=0.03995 -0.07708069 0.010431707 rpy=0.0 0.0 0.0
- joint right_shoulder_yaw: origin xyz=0.0 -0.15135 0.038 rpy=1.5707963267948966 -0.5235993718135523 -3.141592653589793 -> xyz=-0.038 0.0 -0.15135 rpy=0.0 0.0 0.0
- joint right_wrist_pitch: axis 0.0 0.0 -1.0 -> 0.0 1.0 0.0; origin xyz=0.0372391 -0.0215 -0.1665 rpy=-1.5707963267948966 0.0 -2.094395442980787 -> xyz=0.1665 -0.043000007 2.0863829e-08 rpy=0.0 0.0 0.0
- joint right_wrist_roll: axis 0.0 0.0 -1.0 -> 1.0 4.4377618e-18 1.5252148e-08; origin xyz=0.0 -0.12035 0.036 rpy=-1.5707963267948966 -1.047197210609006 0.0 -> xyz=0.12035 -0.036 6.9388939e-18 rpy=0.0 0.0 0.0
- joint right_wrist_yaw: axis 0.0 0.0 -1.0 -> 0.0 0.0 1.0; origin xyz=-0.03315 0.0 -0.043 rpy=-0.0 1.5707963267948966 0.0 -> xyz=0.0 0.043 0.03315 rpy=0.0 0.0 0.0
- joint waist_pitch: axis 0.0 0.0 1.0 -> 0.0 1.0 3.3560631e-09; origin xyz=-0.04275 -0.112 0.05085 rpy=3.141592653589793 -1.5707963267948966 0.0 -> xyz=-0.05085 -0.04275 0.112 rpy=0.0 0.0 0.0
- joint waist_roll: axis 0.0 0.0 -1.0 -> 1.0 0.0 0.0; origin xyz=0.0 -0.00085 0.0 rpy=-1.5707963267948966 0.0 0.0 -> xyz=0.00085 -2.8526536e-12 0.0 rpy=0.0 0.0 0.0
- joint waist_yaw: axis 0.0 0.0 -1.0 -> 0.0 -4.0178666e-17 1.0; origin xyz=0.0 0.056 0.04275 rpy=1.5707963267948966 0.0 0.0 -> xyz=0.0 0.04275 0.056 rpy=0.0 0.0 0.0
